Commit message: Fix in the Crazyflie mass

File: rotors_description/urdf/crazyflie2.xacro (robot description, xacro)
@@ -21,5 +21,5 @@
   <xacro:property name="use_mesh_file" value="true" />
   <xacro:property name="mesh_file" value="package://rotors_description/meshes/crazyflie2.dae" />
-  <xacro:property name="mass" value="0.025" /> <!-- [kg] -->
+  <xacro:property name="mass" value="0.25" /> <!-- [kg] -->
   <xacro:property name="body_width" value="0.045" /> <!-- [m] -->
   <xacro:property name="body_height" value="0.03" /> <!-- [m] -->

Commit message: Bug fixes
Bug fixes in the crazyflie2.xacro file. The saturation values of the hovering controller were updated together with the Omega_e value

File: rotors_description/urdf/crazyflie2.xacro (robot description, xacro)
@@ -21,5 +21,5 @@
   <xacro:property name="use_mesh_file" value="true" />
   <xacro:property name="mesh_file" value="package://rotors_description/meshes/crazyflie2.dae" />
-  <xacro:property name="mass" value="0.25" /> <!-- [kg] -->
+  <xacro:property name="mass" value="0.025" /> <!-- [kg] -->
   <xacro:property name="body_width" value="0.045" /> <!-- [m] -->
   <xacro:property name="body_height" value="0.03" /> <!-- [m] -->
