Commit message: The controller structure has been updated
The controller structure has been updated by splitting the controller into two main files: the upper and low level part. Further details are reported in the changelog files.

File: rotors_description/urdf/component_snippets.xacro (robot description, xacro)
@@ -293,6 +293,6 @@
   <xacro:macro name="imu_plugin_macro"
     params="namespace imu_suffix parent_link imu_topic
-      mass_imu_sensor gyroscope_noise_density gyroscope_random_walk
-      gyroscope_bias_correlation_time gyroscope_turn_on_bias_sigma
+      mass_imu_sensor measurement_divisor measurement_delay gyroscope_noise_density
+      gyroscope_random_walk gyroscope_bias_correlation_time gyroscope_turn_on_bias_sigma
       accelerometer_noise_density accelerometer_random_walk
       accelerometer_bias_correlation_time accelerometer_turn_on_bias_sigma
@@ -321,4 +321,6 @@
         <imuTopic>${imu_topic}</imuTopic> <!-- (string): name of the sensor output topic and prefix of service names (defaults to imu) -->
         <gyroscopeNoiseDensity>${gyroscope_noise_density}</gyroscopeNoiseDensity> <!-- Gyroscope noise density (two-sided spectrum) [rad/s/sqrt(Hz)] -->
+        <measurementDivisor>${measurement_divisor}</measurementDivisor> <!-- only every (seq % measurementDivisor) == 0 measurement is published [int] -->
+        <measurementDelay>${measurement_delay}</measurementDelay> <!-- time that measurement gets held back before it's published in [simulation cycles (int)] -->
         <gyroscopeRandomWalk>${gyroscope_random_walk}</gyroscopeRandomWalk> <!-- Gyroscope bias random walk [rad/s/s/sqrt(Hz)] -->
         <gyroscopeBiasCorrelationTime>${gyroscope_bias_correlation_time}</gyroscopeBiasCorrelationTime> <!-- Gyroscope bias correlation time constant [s] -->
@@ -750,4 +752,6 @@
       parent_link="${namespace}/vi_sensor_link"
       imu_topic="imu"
+      measurement_delay="0"
+      measurement_divisor="1"
       mass_imu_sensor="0.015"
       gyroscope_noise_density="0.0003394"
@@ -770,4 +774,6 @@
       parent_link="${parent_link}"
       imu_topic="ground_truth/imu"
+      measurement_delay="0"
+      measurement_divisor="1"
       mass_imu_sensor="0.00001"
       gyroscope_noise_density="0.0"
@@ -820,4 +826,6 @@
       parent_link="${parent_link}"
       imu_topic="imu"
+      measurement_delay="0"
+      measurement_divisor="1"
       mass_imu_sensor="0.015"
       gyroscope_noise_density="0.0003394"
@@ -833,4 +841,35 @@
     </xacro:imu_plugin_macro>
   </xacro:macro>
+  <xacro:macro name="crazyflie2_odometry" params="namespace parent_link">
+      <xacro:odometry_plugin_macro
+        namespace="${namespace}"
+        odometry_sensor_suffix=""
+        parent_link="${parent_link}"
+        pose_topic="pose"
+        pose_with_covariance_topic="pose_with_covariance"
+        position_topic="position"
+        transform_topic="transform"
+        odometry_topic="odometry"
+        parent_frame_id="world"
+        child_frame_id="${namespace}/base_link"
+        mass_odometry_sensor="0.00001"
+        measurement_divisor="10"
+        measurement_delay="0"
+        unknown_delay="0.0"
+        noise_normal_position="0 0 0"
+        noise_normal_quaternion="0 0 0"
+        noise_normal_linear_velocity="0 0 0"
+        noise_normal_angular_velocity="0 0 0"
+        noise_uniform_position="0 0 0"
+        noise_uniform_quaternion="0 0 0"
+        noise_uniform_linear_velocity="0 0 0"
+        noise_uniform_angular_velocity="0 0 0"
+        enable_odometry_map="false"
+        odometry_map=""
+        image_scale="">
+        <inertia ixx="0.00001" ixy="0.0" ixz="0.0" iyy="0.00001" iyz="0.0" izz="0.00001" /> <!-- [kg m^2] [kg m^2] [kg m^2] [kg m^2] [kg m^2] [kg m^2] -->
+        <origin xyz="0.0 0.0 0.0" rpy="0.0 0.0 0.0" />
+      </xacro:odometry_plugin_macro>
+  </xacro:macro>
   <xacro:macro name="crazyflie2_imu" params="namespace parent_link">
     <!-- Mount an MPU-9250 IMU. -->
@@ -840,4 +879,6 @@
       parent_link="${parent_link}"
       imu_topic="imu"
+      measurement_delay="0"
+      measurement_divisor="2"
       mass_imu_sensor="0.00001"
       gyroscope_noise_density="0.000175"

File: rotors_description/urdf/crazyflie2_base.xacro (robot description, xacro)
@@ -29,4 +29,6 @@
     <xacro:crazyflie2_imu namespace="${namespace}" parent_link="${namespace}/base_link" />
   </xacro:if>
+  <!-- Mount a generic odometry sensor. -->
+  <xacro:crazyflie2_odometry namespace="${namespace}" parent_link="${namespace}/base_link" />
   <xacro:if value="$(arg enable_ground_truth)">
     <xacro:ground_truth_imu_and_odometry namespace="${namespace}" parent_link="${namespace}/base_link" />

Commit message: Make RotorS package compatible with Gazebo9
Make the RotorS package compatible with Gazebo 9. The CrazyS files need to be included and the README.md file update.

File: rotors_description/urdf/component_snippets.xacro (robot description, xacro)
@@ -6,6 +6,4 @@
   Copyright 2015 Janosch Nikolic, ASL, ETH Zurich, Switzerland
   Copyright 2015 Markus Achtelik, ASL, ETH Zurich, Switzerland
-  Copyright 2018 Giuseppe Silano, University of Sannio in Benevento, Italy
-  Copyright 2018 Luigi Iannelli, University of Sannio in Benevento, Italy
   Licensed under the Apache License, Version 2.0 (the "License");
   you may not use this file except in compliance with the License.
@@ -293,6 +291,6 @@
   <xacro:macro name="imu_plugin_macro"
     params="namespace imu_suffix parent_link imu_topic
-      mass_imu_sensor measurement_divisor measurement_delay gyroscope_noise_density
-      gyroscope_random_walk gyroscope_bias_correlation_time gyroscope_turn_on_bias_sigma
+      mass_imu_sensor gyroscope_noise_density gyroscope_random_walk
+      gyroscope_bias_correlation_time gyroscope_turn_on_bias_sigma
       accelerometer_noise_density accelerometer_random_walk
       accelerometer_bias_correlation_time accelerometer_turn_on_bias_sigma
@@ -321,6 +319,4 @@
         <imuTopic>${imu_topic}</imuTopic> <!-- (string): name of the sensor output topic and prefix of service names (defaults to imu) -->
         <gyroscopeNoiseDensity>${gyroscope_noise_density}</gyroscopeNoiseDensity> <!-- Gyroscope noise density (two-sided spectrum) [rad/s/sqrt(Hz)] -->
-        <measurementDivisor>${measurement_divisor}</measurementDivisor> <!-- only every (seq % measurementDivisor) == 0 measurement is published [int] -->
-        <measurementDelay>${measurement_delay}</measurementDelay> <!-- time that measurement gets held back before it's published in [simulation cycles (int)] -->
         <gyroscopeRandomWalk>${gyroscope_random_walk}</gyroscopeRandomWalk> <!-- Gyroscope bias random walk [rad/s/s/sqrt(Hz)] -->
         <gyroscopeBiasCorrelationTime>${gyroscope_bias_correlation_time}</gyroscopeBiasCorrelationTime> <!-- Gyroscope bias correlation time constant [s] -->
@@ -752,6 +748,4 @@
       parent_link="${namespace}/vi_sensor_link"
       imu_topic="imu"
-      measurement_delay="0"
-      measurement_divisor="1"
       mass_imu_sensor="0.015"
       gyroscope_noise_density="0.0003394"
@@ -774,6 +768,4 @@
       parent_link="${parent_link}"
       imu_topic="ground_truth/imu"
-      measurement_delay="0"
-      measurement_divisor="1"
       mass_imu_sensor="0.00001"
       gyroscope_noise_density="0.0"
@@ -826,6 +818,4 @@
       parent_link="${parent_link}"
       imu_topic="imu"
-      measurement_delay="0"
-      measurement_divisor="1"
       mass_imu_sensor="0.015"
       gyroscope_noise_density="0.0003394"
@@ -837,57 +827,4 @@
       accelerometer_bias_correlation_time="300.0"
       accelerometer_turn_on_bias_sigma="0.1960">
-      <inertia ixx="0.00001" ixy="0.0" ixz="0.0" iyy="0.00001" iyz="0.0" izz="0.00001" />
-      <origin xyz="0 0 0" rpy="0 0 0" />
-    </xacro:imu_plugin_macro>
-  </xacro:macro>
-  <xacro:macro name="crazyflie2_odometry" params="namespace parent_link">
-      <xacro:odometry_plugin_macro
-        namespace="${namespace}"
-        odometry_sensor_suffix=""
-        parent_link="${parent_link}"
-        pose_topic="pose"
-        pose_with_covariance_topic="pose_with_covariance"
-        position_topic="position"
-        transform_topic="transform"
-        odometry_topic="odometry"
-        parent_frame_id="world"
-        child_frame_id="${namespace}/base_link"
-        mass_odometry_sensor="0.00001"
-        measurement_divisor="10"
-        measurement_delay="0"
-        unknown_delay="0.0"
-        noise_normal_position="0 0 0"
-        noise_normal_quaternion="0 0 0"
-        noise_normal_linear_velocity="0 0 0"
-        noise_normal_angular_velocity="0 0 0"
-        noise_uniform_position="0 0 0"
-        noise_uniform_quaternion="0 0 0"
-        noise_uniform_linear_velocity="0 0 0"
-        noise_uniform_angular_velocity="0 0 0"
-        enable_odometry_map="false"
-        odometry_map=""
-        image_scale="">
-        <inertia ixx="0.00001" ixy="0.0" ixz="0.0" iyy="0.00001" iyz="0.0" izz="0.00001" /> <!-- [kg m^2] [kg m^2] [kg m^2] [kg m^2] [kg m^2] [kg m^2] -->
-        <origin xyz="0.0 0.0 0.0" rpy="0.0 0.0 0.0" />
-      </xacro:odometry_plugin_macro>
-  </xacro:macro>
-  <xacro:macro name="crazyflie2_imu" params="namespace parent_link">
-    <!-- Mount an MPU-9250 IMU. -->
-    <xacro:imu_plugin_macro
-      namespace="${namespace}"
-      imu_suffix=""
-      parent_link="${parent_link}"
-      imu_topic="imu"
-      measurement_delay="0"
-      measurement_divisor="1"
-      mass_imu_sensor="0.00001"
-      gyroscope_noise_density="0.000175"
-      gyroscope_random_walk="0.0105"
-      gyroscope_bias_correlation_time="1000.0"
-      gyroscope_turn_on_bias_sigma= "0.09"
-      accelerometer_noise_density="0.003"
-      accelerometer_random_walk="0.18"
-      accelerometer_bias_correlation_time="300.0"
-      accelerometer_turn_on_bias_sigma="0.588">
       <inertia ixx="0.00001" ixy="0.0" ixz="0.0" iyy="0.00001" iyz="0.0" izz="0.00001" />
       <origin xyz="0 0 0" rpy="0 0 0" />

Commit message: Add macros for crazyflie's sensors

File: rotors_description/urdf/component_snippets.xacro (robot description, xacro)
@@ -831,4 +831,57 @@
     </xacro:imu_plugin_macro>
   </xacro:macro>
+  <xacro:macro name="crazyflie2_odometry" params="namespace parent_link">
+      <xacro:odometry_plugin_macro
+        namespace="${namespace}"
+        odometry_sensor_suffix=""
+        parent_link="${parent_link}"
+        pose_topic="pose"
+        pose_with_covariance_topic="pose_with_covariance"
+        position_topic="position"
+        transform_topic="transform"
+        odometry_topic="odometry"
+        parent_frame_id="world"
+        child_frame_id="${namespace}/base_link"
+        mass_odometry_sensor="0.00001"
+        measurement_divisor="10"
+        measurement_delay="0"
+        unknown_delay="0.0"
+        noise_normal_position="0 0 0"
+        noise_normal_quaternion="0 0 0"
+        noise_normal_linear_velocity="0 0 0"
+        noise_normal_angular_velocity="0 0 0"
+        noise_uniform_position="0 0 0"
+        noise_uniform_quaternion="0 0 0"
+        noise_uniform_linear_velocity="0 0 0"
+        noise_uniform_angular_velocity="0 0 0"
+        enable_odometry_map="false"
+        odometry_map=""
+        image_scale="">
+        <inertia ixx="0.00001" ixy="0.0" ixz="0.0" iyy="0.00001" iyz="0.0" izz="0.00001" /> <!-- [kg m^2] [kg m^2] [kg m^2] [kg m^2] [kg m^2] [kg m^2] -->
+        <origin xyz="0.0 0.0 0.0" rpy="0.0 0.0 0.0" />
+      </xacro:odometry_plugin_macro>
+  </xacro:macro>
+  <xacro:macro name="crazyflie2_imu" params="namespace parent_link">
+    <!-- Mount an MPU-9250 IMU. -->
+    <xacro:imu_plugin_macro
+      namespace="${namespace}"
+      imu_suffix=""
+      parent_link="${parent_link}"
+      imu_topic="imu"
+      measurement_delay="0"
+      measurement_divisor="1"
+      mass_imu_sensor="0.00001"
+      gyroscope_noise_density="0.000175"
+      gyroscope_random_walk="0.0105"
+      gyroscope_bias_correlation_time="1000.0"
+      gyroscope_turn_on_bias_sigma= "0.09"
+      accelerometer_noise_density="0.003"
+      accelerometer_random_walk="0.18"
+      accelerometer_bias_correlation_time="300.0"
+      accelerometer_turn_on_bias_sigma="0.588">
+      <inertia ixx="0.00001" ixy="0.0" ixz="0.0" iyy="0.00001" iyz="0.0" izz="0.00001" />
+      <origin xyz="0 0 0" rpy="0 0 0" />
+    </xacro:imu_plugin_macro>
+  </xacro:macro>
   <xacro:macro name="default_gps" params="namespace parent_link">
     <!-- Default GPS. -->

Commit message: Delete double pi declaration

File: rotors_description/urdf/component_snippets.xacro (robot description, xacro)
@@ -19,5 +19,4 @@
 -->
 <robot xmlns:xacro="http://ros.org/wiki/xacro">
-  <xacro:property name="pi" value="3.14159265359" />
   <!-- Macro to add logging to a bag file. -->
   <xacro:macro name="bag_plugin_macro"

Commit message: Add ideal IMU sensor

File: rotors_description/urdf/component_snippets.xacro (robot description, xacro)
@@ -6,5 +6,8 @@
   Copyright 2015 Janosch Nikolic, ASL, ETH Zurich, Switzerland
   Copyright 2015 Markus Achtelik, ASL, ETH Zurich, Switzerland
-  Copyright 2018 Giuseppe Silano, University of Sannio in Benevento, Italy
+  Copyright 2020 Ria Sonecha, MIT, USA
+  Copyright 2018 Benjamin Rodriguez, MIT, USA
+  Copyright 2018 Emanuele Aucone, University of Sannio in Benevento
+  Copyright 2020 Giuseppe Silano, University of Sannio in Benevento, Italy
   Copyright 2018 Luigi Iannelli, University of Sannio in Benevento, Italy
   Licensed under the Apache License, Version 2.0 (the "License");
@@ -893,4 +896,26 @@
     </xacro:imu_plugin_macro>
   </xacro:macro>
+  <xacro:macro name="crazyflie2_imuIdeal" params="namespace parent_link">
+  <!-- This is an ideal IMU sensor. -->
+  <xacro:imu_plugin_macro
+    namespace="${namespace}"
+    imu_suffix=""
+    parent_link="${parent_link}"
+    imu_topic="imu"
+    measurement_delay="0"
+    measurement_divisor="1"
+    mass_imu_sensor="0.00001"
+    gyroscope_noise_density="0.0"
+    gyroscope_random_walk="0.0"
+    gyroscope_bias_correlation_time="0.0"
+    gyroscope_turn_on_bias_sigma= "0.0"
+    accelerometer_noise_density="0.0"
+    accelerometer_random_walk="0.0"
+    accelerometer_bias_correlation_time="0.0"
+    accelerometer_turn_on_bias_sigma="0">
+    <inertia ixx="0.00001" ixy="0.0" ixz="0.0" iyy="0.00001" iyz="0.0" izz="0.00001" />
+    <origin xyz="0 0 0" rpy="0 0 0" />
+  </xacro:imu_plugin_macro>
+</xacro:macro>
   <xacro:macro name="default_gps" params="namespace parent_link">
     <!-- Default GPS. -->

File: rotors_description/urdf/crazyflie2.xacro (robot description, xacro)
@@ -1,8 +1,9 @@
 <?xml version="1.0"?>
 <!--
-  Copyright 2018 Giuseppe Silano, University of Sannio in Benevento, Italy
+  Copyright 2020 Giuseppe Silano, University of Sannio in Benevento, Italy
   Copyright 2018 Emanuele Aucone, University of Sannio in Benevento, Italy
   Copyright 2018 Benjamin Rodriguez, MIT, USA
   Copyright 2018 Luigi Iannelli, University of Sannio in Benevento, Italy
+  Copyright 2020 Ria Sonecha, MIT, USA
   Licensed under the Apache License, Version 2.0 (the "License");
   you may not use this file except in compliance with the License.

File: rotors_description/urdf/crazyflie2_base.xacro (robot description, xacro)
@@ -1,8 +1,9 @@
 <?xml version="1.0"?>
 <!--
-  Copyright 2018 Giuseppe Silano, University of Sannio in Benevento, Italy
+  Copyright 2020 Giuseppe Silano, University of Sannio in Benevento, Italy
   Copyright 2018 Emanuele Aucone, University of Sannio in Benevento, Italy
   Copyright 2018 Benjamin Rodriguez, MIT, USA
   Copyright 2018 Luigi Iannelli, University of Sannio in Benevento, Italy
+  Copyright 2020 Ria Sonecha, MIT, USA
   Licensed under the Apache License, Version 2.0 (the "License");
   you may not use this file except in compliance with the License.
@@ -30,4 +31,8 @@
     <xacro:crazyflie2_imu namespace="${namespace}" parent_link="${namespace}/base_link" />
   </xacro:if>
+  <!-- Mount an ideal IMU sensor if the mellinger controller is enabled, otherwise the virtual odometry sensor is used. -->
+  <xacro:if value="$(arg enable_mellinger_controller)">
+    <xacro:crazyflie2_imuIdeal namespace="${namespace}" parent_link="${namespace}/base_link" />
+  </xacro:if>
   <!-- Mount a generic odometry sensor. -->
   <xacro:crazyflie2_odometry namespace="${namespace}" parent_link="${namespace}/base_link" />

Commit message: Changes applied according to #29

File: rotors_description/urdf/component_snippets.xacro (robot description, xacro)
@@ -6,5 +6,8 @@
   Copyright 2015 Janosch Nikolic, ASL, ETH Zurich, Switzerland
   Copyright 2015 Markus Achtelik, ASL, ETH Zurich, Switzerland
-  Copyright 2018 Giuseppe Silano, University of Sannio in Benevento, Italy
+  Copyright 2020 Ria Sonecha, MIT, USA
+  Copyright 2018 Benjamin Rodriguez, MIT, USA
+  Copyright 2018 Emanuele Aucone, University of Sannio in Benevento
+  Copyright 2020 Giuseppe Silano, University of Sannio in Benevento, Italy
   Copyright 2018 Luigi Iannelli, University of Sannio in Benevento, Italy
   Licensed under the Apache License, Version 2.0 (the "License");
@@ -893,4 +896,26 @@
     </xacro:imu_plugin_macro>
   </xacro:macro>
+  <xacro:macro name="crazyflie2_imuIdeal" params="namespace parent_link">
+  <!-- This is an ideal IMU sensor. -->
+  <xacro:imu_plugin_macro
+    namespace="${namespace}"
+    imu_suffix=""
+    parent_link="${parent_link}"
+    imu_topic="imu"
+    measurement_delay="0"
+    measurement_divisor="1"
+    mass_imu_sensor="0.00001"
+    gyroscope_noise_density="0.0"
+    gyroscope_random_walk="0.0"
+    gyroscope_bias_correlation_time="1000.0"
+    gyroscope_turn_on_bias_sigma= "0.0"
+    accelerometer_noise_density="0.0"
+    accelerometer_random_walk="0.0"
+    accelerometer_bias_correlation_time="300.0"
+    accelerometer_turn_on_bias_sigma="0">
+    <inertia ixx="0.00001" ixy="0.0" ixz="0.0" iyy="0.00001" iyz="0.0" izz="0.00001" />
+    <origin xyz="0 0 0" rpy="0 0 0" />
+  </xacro:imu_plugin_macro>
+</xacro:macro>
   <xacro:macro name="default_gps" params="namespace parent_link">
     <!-- Default GPS. -->

Commit message: Add a swarm example with the Crazyflie #44

File: rotors_description/urdf/component_snippets.xacro (robot description, xacro)
@@ -856,5 +856,5 @@
         child_frame_id="${namespace}/base_link"
         mass_odometry_sensor="0.00001"
-        measurement_divisor="10"
+        measurement_divisor="1"
         measurement_delay="0"
         unknown_delay="0.0"

File: rotors_description/urdf/crazyflie2.xacro (robot description, xacro)
@@ -18,5 +18,5 @@
 <robot name="crazyflie2" xmlns:xacro="http://ros.org/wiki/xacro">
   <!-- Properties (Taken from Novel Dynamic Inversion Architecture Design for Quadrocopter Control by Jian Wang et al.) -->
-  <xacro:property name="namespace" value="$(arg mav_name)" />
+  <xacro:property name="namespace" value="$(arg namespace)" />
   <xacro:property name="rotor_velocity_slowdown_sim" value="50" />
   <xacro:property name="use_mesh_file" value="true" />

File: rotors_description/urdf/crazyflie2_base.xacro (robot description, xacro)
@@ -20,5 +20,5 @@
   <!-- Instantiate crazyflie2 "mechanics" -->
   <xacro:include filename="$(find rotors_description)/urdf/crazyflie2.xacro" />
-  <!-- Instantiate a controller. -->
+  <!-- Instantiate a controller.  -->
   <xacro:controller_plugin_macro namespace="${namespace}" imu_sub_topic="imu" />
   <!-- Enable the MAVLink interface. It is useful for the HIL (Hardware-in-the-loop) tests -->
@@ -36,5 +36,5 @@
   </xacro:if>
   <!-- Mount a generic odometry sensor. -->
-  <xacro:crazyflie2_odometry namespace="${namespace}" parent_link="${namespace}/base_link" />
+  <xacro:crazyflie2_odometry namespace="${namespace}" parent_link="${namespace}/base_link"  />
   <!-- Mount a generic odometry sensor employed as ground truth -->
   <xacro:if value="$(arg enable_ground_truth)">
@@ -46,5 +46,6 @@
       namespace="${namespace}"
       bag_file="$(arg log_file)"
-      rotor_velocity_slowdown_sim="${rotor_velocity_slowdown_sim}" />
+      rotor_velocity_slowdown_sim="${rotor_velocity_slowdown_sim}"
+      wait_to_record_bag="$(arg wait_to_record_bag)" />
   </xacro:if>
 </robot>
